File: hardware/tiliqua-motherboard/usbc.kicad_sch (KiCad schematic)
At the start: 9 parts, among them J7 USB_C_Receptacle_USB2.0_14P, U8 TUSB322I, U9 AP2161W

Commit message: * update DNP entries, add nlnet logo
Parts:
- R19: now left out of the parts list
Changed lines of the file:
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@@
 		(unit 1)
 		(exclude_from_sim no)
-		(in_bom yes)
+		(in_bom no)
 		(on_board yes)
 		(dnp yes)
