File: hardware/tiliqua-motherboard/gpdi.kicad_sch (KiCad schematic)
At the start: 12 parts, among them J10 DVI_GPDI, U3 PCA9306DP

Commit message: * update DNP entries, add nlnet logo
Parts:
- R26, R28: now left out of the parts list
Changed lines of the file:
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@@
 		(unit 1)
 		(exclude_from_sim no)
-		(in_bom yes)
+		(in_bom no)
 		(on_board yes)
 		(dnp yes)
@@
 		(unit 1)
 		(exclude_from_sim no)
-		(in_bom yes)
+		(in_bom no)
 		(on_board yes)
 		(dnp yes)

Commit message: * fab 05.01.24
Other:
- note added: "DVI sink == +3V3 with 50ohm series pin_hi == 0mA pin_lo == 3V3 / (50 + 270) ~= 10.3mA (220 adds a bit more headroom than 270, drive strength can be reduced)"
- note removed: "DVI sink == +3V3 with 50ohm series pin_hi == 0mA pin_lo == 3V3 / (50 + 270) ~= 10.3mA (220 adds a bit more headroom, drive strength can be reduced)"
Changed lines of the file:
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@@
 		)
 	)
-	(text "DVI sink == +3V3 with 50ohm series\npin_hi == 0mA\npin_lo == 3V3 / (50 + 270) ~= 10.3mA\n(220 adds a bit more headroom, drive strength can be reduced)"
+	(text "DVI sink == +3V3 with 50ohm series\npin_hi == 0mA\npin_lo == 3V3 / (50 + 270) ~= 10.3mA\n(220 adds a bit more headroom than 270, drive strength can be reduced)"
 		(exclude_from_sim no)
 		(at 92.964 58.928 0)
